File: Electronics/EscornaCPU/2.x/2.40/Escorna_CPU_2_40.brd (EAGLE design)
At the start: 50 x 90.6 mm, 109 parts, among them IC2 ULN2803, IC3 ATMEGA328P-AU, IC4 SX1308, J1 2.54, J2 10118194-0001LF/C, J3 ZL262-4SG, J5 ZL262-4SG, U1 CH340ESMD, U3 ASM1117-5.0, X1 1776275-2, X1.1 1776275-2, Y1 CSTCE16M0V53C-R0

Commit message: Update
Parts:
- added C10, C11: 100nF, Condensatori:C0603-ROUND
- moved R1 0.94 mm to (33.0, 70.8)
- moved XDS1 0.35 mm to (8.38, 71.4)
- moved XDS 0.33 mm to (5.87, 71.4)
Connections:
- net N$11 renamed -D
- net N$14 renamed +D
- net 5V: now also C10.2, C11.2
- net GND: now also C10.1, C11.1
Routing:
- net +D: track 50.5 -> 56.5 mm
- net 5V: track 171.4 -> 174.0 mm, vias 4 -> 12
- net N$15: track 37.6 -> 35.7 mm
- net -D: track 57.2 -> 56.5 mm
- net GND: vias 32 -> 31
Other:
- board text added: "CERN Open Hardware Licence 2.0"
- board text removed: "CERN Open Hardware Licence 1.2 (2.0)"
