File: Electronics/EscornaCPU/2.x/2.40/Escorna_CPU_2_40Amt.brd (EAGLE design)
At the start: 50 x 90.6 mm, 112 parts, among them IC2 ULN2803, IC3 ATMEGA328P-AU, IC4 SX1308, J1 2.54, J2 10118194-0001LF/C, J3 ZL262-4SG, J5 ZL262-4SG, U1 CH340ESMD, U3 ASM1117-5.0, X1 1776275-2, X1.1 1776275-2, Y1 CSTCE16M0V53C-R0

Commit message: Update
Parts:
- removed XDS2: XDESIG, xdesig:XDESIG_CU_2
- moved XDS1 35.6 mm to (26.2, 40.6)
- moved $1_82_$ 9.36 mm to (27.5, 39.4)
Routing:
- net D10: track 62.2 -> 43.7 mm
- net RAW: track 82.9 -> 85.9 mm
- net GND: vias 31 -> 36
Other:
- board text added: "2042"
- board text added: "CPU 2.40.1"
- board text added: "OSHWA ES11"
- board text removed: "2011"
