File: Electronics/EscornaCPU/2.x/2.40/Escorna_CPU_2_40Amt.sch (EAGLE design)
At the start: 101 parts, among them IC2 ULN2803, IC3 ATMEGA328P-AU, IC4 SX1308, J1 2.54, J2 10118194-0001LF/C, J3 ZL262-4SG, J5 ZL262-4SG, U1 CH340ESMD, U3 ASM1117-5.0, X1 1776275-2, X1.1 1776275-2, Y1 CSTCE16M0V53C-R0

Commit message: Update
Parts:
- removed XDS2: XDESIG, xdesig:XDESIG
Other:
- note added: "0021"
- note removed: "002"
- note removed: "Amtega Logo"
Changed lines of the file:
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@@
 <part name="H3" library="holes" deviceset="MOUNT-HOLE" device="3.0" value="3.0"/>
 <part name="H4" library="holes" deviceset="MOUNT-HOLE" device="3.0" value="3.0"/>
-<part name="XDS2" library="xdesig" deviceset="XDESIG" device=""/>
 <part name="ESC" library="escorna" deviceset="ESCORNABOT" device=""/>
 <part name="R19" library="rcl" deviceset="R-EU_" device="0204/7" value="10K"/>
@@
 <text x="246.888" y="17.526" size="1.778" layer="97">XDeSIG</text>
 <text x="173.228" y="25.4" size="2.54" layer="97">PseudoSingularis (PSingularis)  by XDeSIG.</text>
-<text x="254" y="7.62" size="2.54" layer="97">002</text>
+<text x="254" y="7.62" size="2.54" layer="97">0021</text>
 <text x="221.234" y="132.334" size="2.54" layer="95">Enabling LEDs, Default on</text>
 <text x="159.766" y="77.978" size="1.778" layer="97" rot="R270">BUZZ on/off</text>
@@
 <text x="88.646" y="37.338" size="2.54" layer="95" rot="R180">Step-up power</text>
 <text x="75.184" y="4.572" size="1.778" layer="97">MT3608</text>
-<text x="88.9" y="96.52" size="2.54" layer="97" align="center">
-Amtega
-Logo
-</text>
 </plain>
 <instances>
@@
 <instance part="H3" gate="G$1" x="2.54" y="60.96"/>
 <instance part="H4" gate="G$1" x="2.54" y="68.58"/>
-<instance part="XDS2" gate="G$1" x="259.08" y="17.78"/>
 <instance part="ESC" gate="G$1" x="132.08" y="86.36"/>
 <instance part="R19" gate="G$1" x="195.58" y="162.56" rot="R180"/>
